File: gba-umd/gba-umd.kicad_pcb (KiCad board)
At the start: 2 copper layers, 49.5 x 94 mm, 7 parts, among them CON101 HDR2X3, CON102 UMDv3-CONN, CON103 GBA-CONN, U100 MCP23008T-E_SS

Commit message: version 0.1
Routing:
- net /IRQ: track 20.5 -> 12.9 mm, vias 0 -> 1
- net /A19: track 47.1 -> 42.9 mm, vias 1 -> 0
- net /A20: track 41.4 -> 37.9 mm, vias 1 -> 0
- net /A21: track 27.1 -> 24.1 mm, vias 1 -> 2
- net /A18: track 57.5 -> 59.1 mm
- net /A23: track 38.8 -> 37.5 mm, vias 1 -> 0
- net /A22: track 32.7 -> 31.7 mm, vias 1 -> 0
- net GND: vias 0 -> 18
Other:
- board text added: "1"
- board text added: "32"
- board text added: "oxx oxx GBA ID = 0x04 xxo xxo GB ID = 0x05"
- board text removed: "xxo xxo GB ID = 0x05 oxx oxx GBA ID = 0x04"
