File: gba-umd/gba-umd.kicad_sch (KiCad schematic)
At the start: 4 parts, among them U100 MCP23008T-E_SS

Commit message: schematic done
Parts:
- added C101: 0.1uF, db-smt:0603, symbol db-passives:C_0603
- added CON101: HDR2X3, db-thparts:HDR2X3, symbol db-connectors:HDR2X3
- added R101: 10k, db-smt:0603, symbol db-passives:R_0603
Connections:
- net +3V3: now also U100.14 (GP2), U100.20 (Vdd), C101.1, CON101.1, CON101.6; no longer U100.13 (GP1)
- net +5V: now also CON?.34 (+5V), CON?.63 (+5V), CON101.2
- net A16: now also CON?.10 (A16)
- net A17: now also CON?.56 (A17)
- net A18: now also CON?.9 (A18)
- net A19: now also CON?.31 (A19)
- net A20: now also CON?.30 (A20)
- net A21: now also CON?.35 (A21)
- net A22: now also CON?.29 (A22)
- net A23: now also CON?.32 (A23)
- net AD0: now also CON?.14 (D0)
- net AD1: now also CON?.51 (D1)
- net AD10: now also CON?.18 (D10)
- net AD11: now also CON?.47 (D11)
- net AD12: now also CON?.17 (D12)
- net AD13: now also CON?.49 (D13)
- net AD14: now also CON?.15 (D14)
- net AD15: now also CON?.50 (D15)
- net AD2: now also CON?.16 (D2)
- net AD3: now also CON?.48 (D3)
- net AD4: now also CON?.21 (D4)
- net AD5: now also CON?.44 (D5)
- net AD6: now also CON?.20 (D6)
- net AD7: now also CON?.45 (D7)
- net AD8: now also CON?.19 (D8)
- net AD9: now also CON?.46 (D9)
- net GND: now also CON?.33 (GND), CON?.64 (GND), U100.13 (GP1), U100.9 (Vss), C101.2, CON101.5, R101.2; no longer U100.14 (GP2)
- net CARTV: now reaches CON?.1 (3V3)
- net CARTV: now also CON101.4
- net IRQ: now reaches CON?.31 (IRQ)
- net ID: now reaches U100.12 (GP0)
- net ID: now also CON101.3, R101.1
Other:
- note added: "GBA ID = 0x04 GB ID = 0x05"
- note removed: "GBA ID = 0x03 GB ID = 0x04"
- moved on the sheet: CON?, CON?A, U100A, U100B

Commit message: prelim pcb routing
Parts:
- added logo101: dblogo, db-artwork:db-logo_7.5mm, symbol db-artwork:logo
- gave numbers to parts that had none: 2
Connections:
- net +5V: no longer CON102.34 (+5V)
- net IRQ: now also CON102.42 (IO3)
Changed lines of the file:
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@@
-    (stroke (width 0) (type default))
-  )
-  (wire (pts (xy 220.98 127) (xy 231.14 127))
     (stroke (width 0) (type default))
   )
@@
   )
   (wire (pts (xy 69.85 97.79) (xy 82.55 97.79))
+    (stroke (width 0) (type default))
+  )
+  (wire (pts (xy 218.44 106.68) (xy 231.14 106.68))
     (stroke (width 0) (type default))
   )
@@
     (effects (font (size 1.27 1.27)) (justify left bottom))
   )
+  (label "IRQ" (at 218.44 106.68 0) (fields_autoplaced)
+    (effects (font (size 1.27 1.27)) (justify left bottom))
+  )
   (label "CARTV" (at 132.08 50.8 0) (fields_autoplaced)
     (effects (font (size 1.27 1.27)) (justify left bottom))
@@
   (symbol (lib_id "db-vgparts:UMDv3-CONN") (at 236.22 132.08 0) (unit 2)
     (in_bom yes) (on_board yes) (dnp no)
-    (property "Reference" "CON?" (at 236.22 43.18 0)
+    (property "Reference" "CON102" (at 236.22 43.18 0)
       (effects (font (size 1.27 1.27)) (justify left))
     )
@@
       (project "gba-umd"
         (path "/ca61096a-5ed9-48db-a163-e605513173e2"
-          (reference "CON?") (unit 2)
+          (reference "CON102") (unit 2)
         )
       )
@@
   (symbol (lib_id "db-vgparts:GBA-CONN") (at 149.86 48.26 0) (unit 1)
     (in_bom yes) (on_board yes) (dnp no) (fields_autoplaced)
-    (property "Reference" "CON?" (at 156.21 43.18 0)
+    (property "Reference" "CON103" (at 156.21 43.18 0)
       (effects (font (size 1.27 1.27)))
     )
@@
       (project "gba-umd"
         (path "/ca61096a-5ed9-48db-a163-e605513173e2"
-          (reference "CON?") (unit 1)
+          (reference "CON103") (unit 1)
+        )
+      )
+    )
+  )
+  (symbol (lib_id "db-artwork:logo") (at 187.325 151.13 0) (unit 1)
+    (in_bom yes) (on_board yes) (dnp no) (fields_autoplaced)
+    (property "Reference" "logo101" (at 193.04 149.86 0)
+      (effects (font (size 1.524 1.524)) (justify left))
+    )
+    (property "Value" "dblogo" (at 193.04 152.4 0)
+      (effects (font (size 1.524 1.524)) (justify left))
+    )
+    (property "Footprint" "db-artwork:db-logo_7.5mm" (at 187.325 151.13 0)
+      (effects (font (size 1.524 1.524)) hide)
+    )
+    (property "Datasheet" "" (at 187.325 151.13 0)
+      (effects (font (size 1.524 1.524)) hide)
+    )
+    (instances
+      (project "gba-umd"
+        (path "/ca61096a-5ed9-48db-a163-e605513173e2"
+          (reference "logo101") (unit 1)
         )
       )
@@
   (symbol (lib_id "db-vgparts:UMDv3-CONN") (at 64.77 133.35 0) (mirror y) (unit 1)
     (in_bom yes) (on_board yes) (dnp no) (fields_autoplaced)
-    (property "Reference" "CON?" (at 58.42 44.45 0)
+    (property "Reference" "CON102" (at 58.42 44.45 0)
       (effects (font (size 1.27 1.27)))
     )
@@
       (project "gba-umd"
         (path "/ca61096a-5ed9-48db-a163-e605513173e2"
-          (reference "CON?") (unit 1)
+          (reference "CON102") (unit 1)
         )
       )
@@
         )
       )
-    )
-  )
-  (symbol (lib_id "power:+5V") (at 220.98 127 90) (mirror x) (unit 1)
-    (in_bom yes) (on_board yes) (dnp no)
-    (property "Reference" "#PWR0109" (at 224.79 127 0)
-      (effects (font (size 1.27 1.27)) hide)
-    )
-    (property "Value" "+5V" (at 213.36 127 90)
-      (effects (font (size 1.27 1.27)) (justify right))
-    )
-    (property "Footprint" "" (at 220.98 127 0)
-      (effects (font (size 1.27 1.27)) hide)
-    )
-    (property "Datasheet" "" (at 220.98 127 0)
-      (effects (font (size 1.27 1.27)) hide)
-    )
-    (pin "1")
-    (instances
-      (project "gba-umd"
-        (path "/ca61096a-5ed9-48db-a163-e605513173e2"
-          (reference "#PWR0109") (unit 1)
-        )
-      )

Commit message: version 0.1
Other:
- title: GBA UMDv3 Cartridge Adapter -> GB/GBA UMDv3 Cartridge Adapter
- moved on the sheet: C101, CON101, CON102A, CON102B, CON103, R101, U100A, U100B
